Commit message: Rebase from 'debian/kinetic/create_description'

File: urdf/create.urdf.xacro (robot description, xacro)
@@ -3,6 +3,6 @@
   <!-- Macro for TurtleBot body. Including Gazebo extensions, but does not include Kinect -->
   <xacro:include filename="$(find create_description)/urdf/create_gazebo.urdf.xacro"/>
-  <property name="base_x" value="0.33" />
-  <property name="base_y" value="0.33" />
+  <xacro:property name="base_x" value="0.33" />
+  <xacro:property name="base_y" value="0.33" />
 	  <xacro:macro name="create">
 	    <material name="Green">
@@ -41,5 +41,5 @@
 	      <origin xyz="0.0 0.0 0.0308" rpy="0 0 0" />
 	      <geometry>
-	        <cylinder length="0.0611632" radius="0.016495"/>
+	        <cylinder length="0.0611632" radius="0.16495"/>
 	      </geometry>
 	    </collision>
